File: hardware/esp8266ex-tryout.kicad_pcb (KiCad board)
At the start: 2 copper layers, 20 parts, among them U1 ESP8266EX, U2 W25Q32JVSSIQ, Y1 O_26M,3225

Commit message: update,
Routing:
- net Vesp8266: track 28.3 -> 69.6 mm, vias 7 -> 6
- net GND: track 34.5 -> 66.9 mm, vias 1 -> 3
- net Net-(C1-Pad2): track 0.00 -> 14.4 mm, vias 0 -> 1
- net /SD_D2: track 0.00 -> 12.9 mm, vias 0 -> 2
- net /SD_D1: track 0.00 -> 12.9 mm, vias 0 -> 2
- net /SD_CMD: track 0.00 -> 6.95 mm, vias 0 -> 2
- net Net-(R2-Pad2): track 0.00 -> 6.27 mm, vias 0 -> 1
- net Net-(C2-Pad2): track 0.00 -> 4.84 mm, vias 0 -> 1
- net /SD_CLK: track 0.00 -> 4.04 mm, vias 0 -> 1
- net /SD_D3: track 0.00 -> 3.88 mm
- net /SD_D0: track 0.00 -> 3.49 mm
- net Net-(R1-Pad2): track 0.00 -> 2.88 mm
- net /GPIO14: track 1.46 -> 2.32 mm

Commit message: update to add debug ,
Parts:
- added U3: ESP8266EX_SERVICE, footprint-lib:ESP8266EX_SERVICE, F.Cu at (60.1, 20.0)
- moved Y1 1.14 mm to (48.7, 19.3)
- moved C1 1.14 mm to (50.0, 19.3)
- moved C2 1.14 mm to (47.3, 19.3)
- moved R1 0.91 mm to (43.0, 20.4)
Routing:
- net /RST: track 0.00 -> 30.7 mm, vias 0 -> 3
- net GND: track 66.9 -> 85.7 mm, vias 3 -> 4
- net /UTXD: track 0.00 -> 17.5 mm
- net /URXD: track 0.00 -> 16.8 mm
- net Net-(C2-Pad2): track 4.84 -> 6.02 mm
- net Net-(R1-Pad2): track 2.88 -> 3.92 mm
- net Net-(C1-Pad2): track 14.4 -> 14.9 mm
- net Vesp8266: vias 6 -> 5

Commit message: update for RN,
Parts:
- added RN1: RN_201,0603, Resistor_SMD:R_Array_Concave_4x0603, F.Cu at (49.1, 24.7)
- added RN2: RN_201,0603, Resistor_SMD:R_Array_Concave_4x0603, F.Cu at (49.1, 28.7)
- moved U3 6.77 mm to (53.5, 18.5), turned to 90 degrees
- moved R2 5.41 mm to (57.2, 28.5)
- moved C7 5.41 mm to (57.8, 24.9)
- moved U2 5.41 mm to (57.8, 26.6)
Connections:
- U1 pad 18: /SD_D2 -> Net-(RN2-Pad6)
- U1 pad 19: /SD_D3 -> Net-(RN2-Pad5)
- U1 pad 20: /SD_CMD -> Net-(RN1-Pad8)
- U1 pad 21: Net-(R2-Pad2) -> Net-(RN1-Pad7)
- U1 pad 22: /SD_D0 -> Net-(RN1-Pad6)
- U1 pad 23: /SD_D1 -> Net-(RN1-Pad5)
Routing:
- net /SD_CLK: track 4.04 -> 19.8 mm, vias 1 -> 3
- net Net-(R2-Pad2): track 6.27 -> 0.00 mm, vias 1 -> 0
- net /SD_D1: track 12.4 -> 18.4 mm, vias 2 -> 0
- net /SD_D0: track 3.49 -> 9.22 mm, vias 0 -> 2
- net Net-(RN1-Pad5): track 0.00 -> 4.32 mm
- net Net-(RN1-Pad6): track 0.00 -> 4.02 mm
- net /SD_D3: track 3.88 -> 7.84 mm
- net GND: track 85.7 -> 82.1 mm, vias 4 -> 3
- net Net-(RN1-Pad7): track 0.00 -> 3.58 mm
- net Net-(RN2-Pad6): track 0.00 -> 3.35 mm
- net Net-(RN1-Pad8): track 0.00 -> 3.18 mm
- net Net-(RN2-Pad5): track 0.00 -> 2.87 mm
- net /UTXD: track 17.5 -> 15.4 mm
- net /SD_CMD: track 6.95 -> 4.90 mm, vias 2 -> 0
- net /RST: track 30.7 -> 28.6 mm, vias 3 -> 2
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